File: Antenna_Impedance_Match/Antenna_Impedance_Match.kicad_pcb (KiCad board)
At the start: 2 copper layers, 30 x 15 mm, 5 parts, among them J1 Conn_Coaxial, J2 Conn_Coaxial

Commit message: More work, esp on firmware
Parts:
- removed J2: Conn_Coaxial, Repowered_Connectors:Cinch_VF320
- added TP2: TestPoint, TestPoint:TestPoint_Bridge_Pitch3.81mm_Drill1.3mm, F.Cu at (153.1, 81.9)
- C1: value 6.8pF -> 18pF; footprint Capacitor_SMD:C_0603_1608Metric -> Capacitor_SMD:C_0805_2012Metric
- C2: footprint Capacitor_SMD:C_0603_1608Metric -> Capacitor_SMD:C_0805_2012Metric
- L1: value 47nH -> 68nH; footprint Repowered_Inductors_SMD:L_Coilcraft_1111SQ-47N -> Repowered_Inductors_SMD:L_Coilcraft_1515SQ-68N
- moved C2 4.70 mm to (144.5, 81.0), turned to 90 degrees
- moved L1 2.45 mm to (138.8, 80.0)
- moved C1 0.43 mm to (133.3, 81.0), turned to 90 degrees
Connections:
- C1 pad 1: /RF_50_SE -> GND
- C1 pad 2: GND -> /RF_50_SE
- C2 pad 1: /RF_75_SE -> GND
- C2 pad 2: GND -> /RF_75_SE
Routing:
- net GND: track 0.00 -> 9.28 mm, vias 42 -> 43
Other:
- board size 30 x 15 mm -> 30 x 14 mm
- board text added: "(C) 2023 ADAM CORDINGLEY"
- board text added: "acordingley.us/ke8itf"
