File: Antenna_Impedance_Match/Antenna_Impedance_Match.kicad_sch (KiCad schematic)
At the start: 5 parts, among them J1 Conn_Coaxial, J2 Conn_Coaxial

Commit message: More work, esp on firmware
Parts:
- removed C1: 6.8pF, Capacitor_SMD:C_0603_1608Metric, symbol Device:C
- removed C2: 18pF, Capacitor_SMD:C_0603_1608Metric, symbol Device:C
- removed J2: Conn_Coaxial, Repowered_Connectors:Cinch_VF320, symbol Connector:Conn_Coaxial
- added C5 (x2): 18pF, Capacitor_SMD:C_0805_2012Metric, symbol Device:C
- added TP2: TestPoint, TestPoint:TestPoint_Bridge_Pitch3.81mm_Drill1.3mm, symbol Connector:TestPoint
- L5: value 47nH -> 68nH; footprint Repowered_Inductors_SMD:L_Coilcraft_1111SQ-47N -> Repowered_Inductors_SMD:L_Coilcraft_1515SQ-68N
Connections:
- net GND: now also C5.1, C5.1, TP2.1
- net RF_50_SE: now also C5.2
- net RF_75_SE: now also C5.2
