File: Weather_Balloon_Payload_HW/Weather_Balloon_Payload_HW.kicad_pcb (KiCad board)
At the start: 4 copper layers, 100 x 90 mm, 249 parts, among them J1 Conn_01x02, J10 Conn_01x02, J2 Conn_01x08, J3 Conn_01x04, J4 Conn_01x04, J5 MM8430-2610, J6 MM8430-2610, J7 MM8430-2610, J8 Conn_Coaxial, J9 XKTF-015-G, Q1 Si2302, Q2 Si2301, Q3 Si2302, Q4 Si2301, Q5 Si2302, T1 CX2045LNLT, T2 TC2-72T+, T3 TC2-72T+, U1 AP3211K, U10 PGA-105, U11 PGA-105, U12 TLV9061, U13 MAX2606, U14 TS5A3159ADBVR, U15 ADA4891-1, U16 PGA-105, U17 PHA13-HLN+, U2 AP3211K, U3 ADP1612, U4 NCP308SN180T1G, U5 MAX-M8C, U6 MS5607-02BA, U7 MCP9808_DFN, U8 STM32F334C8Tx, U9 ADF4002BRUZ, Y1 12MHz

Commit message: Add fabrication files
Parts:
- removed U7: MCP9808_DFN, Package_DFN_QFN:DFN-8-1EP_3x2mm_P0.5mm_EP1.7x1.4mm
- added C91: 18pF, Capacitor_SMD:C_0402_1005Metric, F.Cu at (203.0, 73.3)
- added C92: 18pF, Capacitor_SMD:C_0402_1005Metric, F.Cu at (202.8, 68.0)
- added G***: LOGO, silk_imgs:silk_imgs, B.Cu at (196.4, 85.7)
- added J11: MM8430-2610, Repowered_Connectors:Connector_Murata_MM8430-2610RA1, F.Cu at (141.2, 95.0)
- added J12: MM8430-2610, Repowered_Connectors:Connector_Murata_MM8430-2610RA1, F.Cu at (145.4, 102.4)
- added L15: 68nH, Repowered_Inductors_SMD:L_Coilcraft_1515SQ-68N, F.Cu at (199.0, 70.9)
- added U18: MCP9808_MSOP, Package_SO:MSOP-8_3x3mm_P0.65mm, F.Cu at (152.0, 135.7)
- C66, C73: value 12.5pF -> 12pF
- L14: footprint Repowered_Inductors_SMD:L_Coilcraft_1111SQ-39N -> Repowered_Inductors_SMD:L_Coilcraft_1111SQ-47N
- moved C87 10.3 mm to (193.6, 73.8), turned to -90 degrees
- moved C86 10.1 mm to (193.1, 66.4), turned to 180 degrees
- moved L14 9.23 mm to (193.6, 69.5)
- moved C83 6.27 mm to (194.1, 65.0), turned to 0 degrees
- moved TP10 2.80 mm to (129.0, 92.6)
- moved C60 1.75 mm to (141.7, 88.4)
- moved C61 1.75 mm to (145.0, 88.6)
- moved C62 1.75 mm to (133.9, 88.9)
- moved C63 1.75 mm to (136.2, 85.1)
- moved C64 1.75 mm to (128.4, 88.7)
- moved C65 1.75 mm to (132.2, 89.3)
- moved C88 1.75 mm to (138.9, 92.0)
- moved L7 1.75 mm to (130.1, 85.9)
- moved R50 1.75 mm to (143.3, 85.1)
- moved R51 1.75 mm to (136.2, 88.9)
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Connections:
- C87 pad 1: /Transmitter/ANT_CONN -> /Transmitter/ANT_MATCH_2
- L14 pad 2: /Transmitter/ANT_CONN -> /Transmitter/ANT_MATCH_2
- U8 pad 25: PWM_SIGNAL -> /Microcontroller/HRTIM_CHC1
Routing:
- net PA_EN: track 5.11 -> 90.6 mm, vias 0 -> 2
- net I2C_SCL: track 44.7 -> 130.1 mm, vias 1 -> 5
- net I2C_SDA: track 50.5 -> 128.1 mm, vias 1 -> 5
- net GPS_PPS: track 0.00 -> 66.3 mm, vias 0 -> 2
- net GPS_EXTINT: track 0.00 -> 65.4 mm, vias 0 -> 2
- net 5P0_EN: track 5.11 -> 69.9 mm, vias 0 -> 4
- net UART_GPS_MCU: track 5.45 -> 52.8 mm, vias 1 -> 2
- net UART_MCU_GPS: track 5.28 -> 52.3 mm, vias 1 -> 2
- net SPI_MOSI: track 18.0 -> 63.0 mm, vias 1 -> 2
- net PLL_LE: track 10.5 -> 51.9 mm, vias 2 -> 3
- net PLL_CE: track 4.43 -> 44.9 mm, vias 0 -> 2
- net SPI_SCLK: track 19.9 -> 59.8 mm, vias 2 -> 5
- net +8V: track 58.3 -> 19.0 mm
- net TSNS_EXT_ALERT: track 8.55 -> 41.6 mm, vias 1 -> 3
- net /Power/UVLO_RSTB: track 24.5 -> 55.5 mm, vias 4 -> 5
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- added copper zone on In2.Cu, net +3V0
- added copper zone on B.Cu, net +5V
- added copper zone on In2.Cu, net +8V
- removed copper zone on B.Cu, net +8V
Other:
- outline, holes or cut-outs redrawn
- board text added: "FSK IN"
- board text added: "FSK OUT"
- board text added: "HIGH-ALTITUDE BALLOON PAYLOAD REV 1.0 (C) 2023 ADAM CORDINGLEY KE8ITF http://acordingley.us/ke8itf/"
