File: Weather_Balloon_Payload_HW/transmitter.kicad_sch (KiCad schematic)
At the start: 52 parts, among them J5 MM8430-2610, J8 Conn_Coaxial, T2 TC2-72T+, T3 TC2-72T+, U11 PGA-105, U11 PHA13-HLN+, U15 ADA4891-1

Commit message: Update README, block diagrams, schem. Begin layout
Parts:
- removed C1 (x2): 47pF, Capacitor_SMD:C_0402_1005Metric, symbol Device:C
- removed C1 (x2): 1.0pF, Capacitor_SMD:C_0402_1005Metric, symbol Device:C
- removed L5 (x2): 82nH, Inductor_SMD:L_1008_2520Metric, symbol Device:L
- added C1 (x2): 110pF, Capacitor_SMD:C_0402_1005Metric, symbol Device:C
- added C1 (x2): 10pF, Capacitor_SMD:C_0402_1005Metric, symbol Device:C
- added C1: 4.7pF, Capacitor_SMD:C_0402_1005Metric, symbol Device:C
- added C54: 100pF, Capacitor_SMD:C_0402_1005Metric, symbol Device:C
- added L5: 47nH, Repowered_Inductors_SMD:L_Coilcraft_1111SQ-39N, symbol Device:L
- added L5: 180nH, Repowered_Inductors_SMD:L_Coilcraft_2222SQ-181, symbol Device:L
- added L5: 120nH, Inductor_SMD:L_1008_2520Metric_Pad1.43x2.20mm_HandSolder, symbol Device:L
- added TP1: TestPoint, TestPoint:TestPoint_Pad_D1.0mm, symbol Connector:TestPoint
- C1: value 3.9pF -> 12.5pF
- C1: value 1.0pF -> 4.7pF; JLCPCB Part # C277493 -> (none); Manufacturer YAGEO -> (none); Mfr. Part # CC0402CRNPO9BN1R0 -> (none)
- C1: value 47pF -> 110pF
Connections:
- net ANT_CONN: now also C1.1, L5.2; no longer C83.1
- net BASEBAND: now also C54.2
- net DBM_1: now also T2.3; no longer T2.1
- net DBM_3: now also T2.1; no longer T2.3
- net GND: now also T2.6, C1.2, C1.2, C1.2, C1.2; no longer T2.4
- net LO_OUT: now also T2.4; no longer T2.6
- net MIX_FILT_2: now also C1.1, C1.2
- net MIX_FILT_3: now also C1.1, C1.1
- net PA_RF_DC: now also L5.2
- net PWM_SIGNAL: now also TP1.1
- net RF_TX_AMP_OUT: now also L5.2
- net U15_INN: now also C54.1
- net V-8P0_PA: now also L5.1
- net at C43.1, C75.2, R41.1: now also L5.1
- new net ANT_MATCH: C1.1, C83.1, L5.1
Other:
- note added: "4.9MHz LPF"
- note added: "~330MHz LPF"
- moved on the sheet: C1, D6, D7, D8, D9, J5, J8, L10, L7, L8, L9, R13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

Commit message: Add fabrication files
Parts:
- added C28 (x2): 18pF, Capacitor_SMD:C_0402_1005Metric, symbol Device:C
- added L5: 68nH, Repowered_Inductors_SMD:L_Coilcraft_1515SQ-68N, symbol Device:L
- C1: value 12.5pF -> 12pF; JLCPCB Part # (none) -> C161305; Manufacturer (none) -> Murata Electronics; Mfr. Part # (none) -> GJM1555C1H120GB01D
- C1: JLCPCB Part # (none) -> C85856; Manufacturer (none) -> Murata Electronics; Mfr. Part # (none) -> GCM1555C1H4R7CA16D
- C1: JLCPCB Part # (none) -> C185562; Manufacturer (none) -> Murata Electronics; Mfr. Part # (none) -> GRM1555C1H111JA01D
- C1: JLCPCB Part # (none) -> C76951; Manufacturer (none) -> Murata Electronics; Mfr. Part # (none) -> GRM1555C1H151JA01D
- C1: JLCPCB Part # (none) -> C161145; Manufacturer (none) -> Murata Electronics; Mfr. Part # (none) -> GCM1555C1H100FA16D
- L5: footprint Repowered_Inductors_SMD:L_Coilcraft_1111SQ-39N -> Repowered_Inductors_SMD:L_Coilcraft_1111SQ-47N
- R13: JLCPCB Part # (none) -> C423191; Manufacturer (none) -> UNI-ROYAL(Uniroyal Elec); Mfr. Part # (none) -> 0402WGF3240TCE
- R13: JLCPCB Part # (none) -> C102889; Manufacturer (none) -> RALEC; Mfr. Part # (none) -> RTT022200FTH
- R7: JLCPCB Part # (none) -> C144726; Manufacturer (none) -> YAGEO; Mfr. Part # (none) -> AC0402JR-071K5L
Connections:
- net ANT_CONN: now also C28.2, L5.2; no longer C1.1, L5.2
- net GND: now also C28.1, C28.1
- new net ANT_MATCH_2: C1.1, C28.2, L5.1, L5.2
Other:
- note added: "50Ohm ~ 75Ohm"
- moved on the sheet: J8
